File: PCB/PCB_Eagle_mit_VCNL/Robot_Psoc.brd (EAGLE design)
At the start: 235.3 x 59.5 mm, 178 parts, among them IC1 LD117AS33TR, U1 CY8C4247AZI-M485, U2 VCNL4010-GS08, U3 VCNL4010-GS08, U4 VCNL4010-GS08, U5 VCNL4010-GS08, X1 FH12-10S-0.5SH, X2 FH12-10S-0.5SH

Commit message: 15/11/2016
Parts:
- added CANH_3_C2, CANH_4_C2, CANL_3_C2, CANL_4_C2, GND_3_C2, GND_4_C2, VCC_3_C2, VCC_4_C2: TPB2,54, testpad:B2,54
Connections:
- net GND_C2: now also GND_3_C2.TP, GND_4_C2.TP
- net N$32: now also CANL_3_C2.TP, CANL_4_C2.TP
- net N$7: now also CANH_3_C2.TP, CANH_4_C2.TP
- net VCC_C2: now also VCC_3_C2.TP, VCC_4_C2.TP
Routing:
- net 3V3_C2: track 167.6 -> 216.1 mm
- net N$32: track 111.1 -> 153.3 mm
- net N$7: track 110.0 -> 150.0 mm
- net GND_C2: track 193.0 -> 230.1 mm, vias 5 -> 7
- net VCC_C2: track 113.3 -> 136.2 mm, vias 2 -> 5
