File: PCB/PCB_Eagle_mit_Xbee_Adapter_Robot/Xbee_Adapter.sch (EAGLE design)
At the start: 186 parts, among them IC1 LD117AS33TR, U1 CY8C4247AZI-M485, U2 VCNL4010-GS08, U3 VCNL4010-GS08, U4 VCNL4010-GS08, U5 VCNL4010-GS08, X1 FH12-10S-0.5SH, X2 FH12-10S-0.5SH

Commit message: 15 de Enero de 2017
Xbee Adapter Agregado
Parts:
- removed 3V3_C1, 3V3_C2, 3V3_C2_C3, 3V3_C3, CANH_C1, CANH_C2, CANH_C2_C3, CANH_C3, CANL_C1, CANL_C2, CANL_C2_C3, CANL_C3, DN_C1, DN_C2, GND_C1, GND_C2, GND_C2_C3, GND_C3, L_C1_C3, L_C1_C4, L_C2, L_C2_C1, L_C2_C3, L_C2_C4, L_C3, L_C3_C2, L_C4, L_C4_C1, MECH_LINK_1, MECH_LINK_11, MECH_LINK_2, MECH_LINK_3, MECH_LINK_4, MECH_LINK_5, MECH_LINK_6, MECH_LINK_7, MECH_LINK_8, MECH_LINK_9, SCL_S2_C2, SCL_S2_C2_C1, SCL_S3_C1_C3, SCL_S3_C3, SCL_S3_C3_C1, SCL_S3_C3_C2, SCL_S4_C1_C4, SCL_S4_C4, SCL_S4_C4_C1, SCL_S4_C4_C2, SDA_S2_C1, SDA_S2_C2_C2, SDA_S3_C1, SDA_S3_C1_C1, SDA_S3_C3_C3, SDA_S3_C3_C4, SDA_S4_C1, SDA_S4_C1_C1, SDA_S4_C4_C3, SDA_S4_C4_C4, VCC_C1, VCC_C2, VCC_C2_C3, VCC_C3, VDDA_C1, VDDA_C2, VDDD_C1, VDDD_C2, VDDIO_C1, VDDIO_C2: PTR1TP11R, testpad:PTR1TP11R
- removed CANH_1_C2, CANH_1_C3, CANH_1_C4, CANH_2_C1, CANH_2_C2, CANH_2_C3, CANH_2_C4, CANH_3_C1, CANH_3_C2, CANH_3_C3, CANH_3_C4, CANH_4_C1, CANH_4_C2, CANH_4_C3, CANH_4_C4, CANL_1_C2, CANL_1_C3, CANL_1_C4, CANL_2_C1, CANL_2_C2, CANL_2_C3, CANL_2_C4, CANL_3_C1, CANL_3_C2, CANL_3_C3, CANL_3_C4, CANL_4_C1, CANL_4_C2, CANL_4_C3, CANL_4_C4, GND_1_C2, GND_1_C3, GND_1_C4, GND_2_C1, GND_2_C2, GND_2_C3, GND_2_C4, GND_3_C1, GND_3_C2, GND_3_C3, GND_3_C4, GND_4_C1, GND_4_C2, GND_4_C3, GND_4_C4, VCC_1_C1, VCC_1_C2, VCC_1_C3, VCC_1_C4, VCC_2_C2, VCC_2_C3, VCC_2_C4, VCC_3_C1, VCC_3_C2, VCC_3_C3, VCC_3_C4, VCC_4_C1, VCC_4_C2, VCC_4_C3, VCC_4_C4: TPB2,54, testpad:TPB2,54
- removed DINA: (no value), pinhead:PINHD-1X3
- removed LED1, LED2, LED3, LED4, LED5: (no value), adafruit:LEDCHIPLED_0805
- removed R10, R12, R24, R25, R26, R27, R6, R8: 4.7k, rcl:R-EU_R0805
- removed R19, R20, R21, R22, R23, R4, R5, R7, R9: 220, rcl:R-EU_R0805
- removed S1: SWS002, smd-special:SWS002
- removed U2, U3, U4, U5: VCNL4010-GS08, VCNL4010-GS08:VCNL4010-GS08
- removed X2: FH12-10S-0.5SH, con-hirose2:FH12-10S-0.5SH
- added XB1: XBEE, xbee:XBEE
- X1: value FH12-10S-0.5SH -> (none); device con-hirose2:FH12-10S-0.5SH -> con-wago-508:W237-02P
Connections:
- removed net 3V3_C1: 3V3_C1.TP, CN1.VBUS, R14.1, R6.1, R8.1, U$1.VCC, U2.IR_AN, U2.VDD
- removed net 3V3_C2: 3V3_C2.TP, 3V3_C2_C3.TP, IC1.OUT, L1.1, L2.1, LED5.A, R10.1, R12.1, R15.1, U3.IR_AN, U3.VDD
- removed net 3V3_C3: 3V3_C3.TP, R26.2, R27.2, U4.IR_AN, U4.VDD, X1-5.1
- removed net 3V3_C4: R24.2, R25.2, U5.IR_AN, U5.VDD, X2-5.1
- removed net CANH_C3: CANH_1_C3.TP, CANH_2_C3.TP, CANH_3_C3.TP, CANH_4_C3.TP, CANH_C3.TP, X1-4.1
- removed net CANH_C4: CANH_1_C4.TP, CANH_2_C4.TP, CANH_3_C4.TP, CANH_4_C4.TP, X2-4.1
- removed net CANL_C3: CANL_1_C3.TP, CANL_2_C3.TP, CANL_3_C3.TP, CANL_4_C3.TP, CANL_C3.TP, X1-3.1
- removed net CANL_C4: CANL_1_C4.TP, CANL_2_C4.TP, CANL_3_C4.TP, CANL_4_C4.TP, X2-3.1
- removed net GND3: GND_1_C3.TP, GND_2_C3.TP, GND_3_C3.TP, GND_4_C3.TP, GND_C3.TP, R21.2, R7.1, U4.GND@1, U4.GND@2, X1-2.1, X1-6.1
- removed net GND4: GND_1_C4.TP, GND_2_C4.TP, GND_3_C4.TP, GND_4_C4.TP, R22.2, R9.1, U5.GND@1, U5.GND@2, X2-2.1, X2-6.1
- removed net GND_C1: C10.2, C4.2, C5.2, C6.2, C7.2, C8.2, C9.2, CN1.D-, GND_1_C1.TP, GND_2_C1.TP, GND_3_C1.TP, GND_4_C1.TP, GND_C1.TP, R13.1, R17.2, R18.1, R19.2, R4.2, U$1.GND, U1.VSSA1, U1.VSSA2, U1.VSSD, U1.VSSIO, U2.GND@1, U2.GND@2
- removed net GND_C2: DINA.3, GND_1_C2.TP, GND_2_C2.TP, GND_3_C2.TP, GND_4_C2.TP, GND_C2.TP, GND_C2_C3.TP, IC1.ADJ, R20.2, R23.2, R5.1, U3.GND@1, U3.GND@2
- removed net LED_S1: LED1.A, U1.P2.2
- removed net LED_S2: L_C2.TP, U1.P2.3
- removed net LED_S2_C2: LED2.A, L_C2_C1.TP
- removed net LED_S3: L_C3.TP, U1.P2.4
- removed net LED_S3_C3: LED3.A, L_C2_C3.TP
- removed net LED_S4: L_C4.TP, U1.P2.5
- removed net LED_S4_C4: LED4.A, X2-9.1
- removed net LED_T_S4: L_C2_C4.TP, X1-9.1
- removed net MOTOR: S1.3, U1.P2.6, U1.P2.7
- removed net N$10: SDA_S3_C1_C1.TP, SDA_S3_C3_C3.TP
- removed net N$13: DN_C1.TP, S1.2
- removed net N$14: LED1.C, R19.1
- removed net N$15: LED2.C, R20.1
- removed net N$16: LED3.C, R21.1
- removed net N$17: LED4.C, R22.1
- removed net N$18: LED5.C, R23.1
- removed net N$19: DINA.1, DN_C2.TP
- removed net N$20: L_C1_C4.TP, L_C4_C1.TP
- removed net N$21: R4.1, U2.IR_CA@1, U2.IR_CA@2
- removed net N$22: L_C1_C3.TP, L_C3_C2.TP
- removed net N$26: SCL_S3_C1_C3.TP, SCL_S3_C3_C1.TP
- removed net N$27: SCL_S4_C1_C4.TP, SCL_S4_C4_C1.TP
- removed net N$29: VCC_1_C1.TP, VCC_2_C1.TP, VCC_3_C1.TP, VCC_4_C1.TP, VCC_C1.TP
- removed net N$32: CANL_1_C2.TP, CANL_2_C2.TP, CANL_3_C2.TP, CANL_4_C2.TP, CANL_C2.TP, CANL_C2_C3.TP
- removed net N$43: R5.2, U3.IR_CA@1, U3.IR_CA@2
- removed net N$44: SDA_S4_C1_C1.TP, SDA_S4_C4_C3.TP
- removed net N$46: R9.2, U5.IR_CA@1, U5.IR_CA@2
- removed net N$5: R16.2, S1.4, U$1.CANH
- removed net N$7: CANH_1_C2.TP, CANH_2_C2.TP, CANH_3_C2.TP, CANH_4_C2.TP, CANH_C2.TP, CANH_C2_C3.TP
- removed net N$8: R7.2, U4.IR_CA@1, U4.IR_CA@2
- removed net SCL_S1: R8.2, U1.P2.0/SCB1:SCL1, U2.SCL
- removed net SCL_S2_U: R10.2, SCL_S2_C2_C1.TP, U3.SCL
- removed net SCL_S3_U: R27.1, SCL_S3_C3_C2.TP, U4.SCL
- removed net SCL_S4: SCL_S4_C4.TP, U1.P1.0
- removed net SCL_S4_U: SCL_S4_C4_C2.TP, X1-7.1
- removed net SCL_S4_U_1: R25.1, U5.SCL, X2-7.1
- removed net SDA_S1: R6.2, U1.P2.1/SCB1:SDA1, U2.SDA
- removed net SDA_S2_U: R12.2, SDA_S2_C2_C2.TP, U3.SDA
- removed net SDA_S3_U: R26.1, SDA_S3_C3_C4.TP, U4.SDA
- removed net SDA_S4: SDA_S4_C1.TP, U1.P1.1
- removed net SDA_S4_U: SDA_S4_C4_C4.TP, X1-8.1
- removed net SDA_S4_U_1: R24.1, U5.SDA, X2-8.1
- removed net VCC_C2: DINA.2, IC1.IN, VCC_1_C2.TP, VCC_2_C2.TP, VCC_3_C2.TP, VCC_4_C2.TP, VCC_C2.TP, VCC_C2_C3.TP
- removed net VCC_C3: VCC_1_C3.TP, VCC_2_C3.TP, VCC_3_C3.TP, VCC_4_C3.TP, VCC_C3.TP, X1-1.1, X1-10.1
- removed net VCC_C4: VCC_1_C4.TP, VCC_2_C4.TP, VCC_3_C4.TP, VCC_4_C4.TP, X2-1.1, X2-10.1
- removed net VDDA2: L1.2, VDDA_C2.TP
- removed net VDDD2: L2.2, VDDD_C2.TP
- removed net VDDIO2: R15.2, VDDIO_C2.TP
- new net 3V3: CN1.VBUS, IC1.OUT, L1.1, L2.1, R14.1, R15.1, U$1.VCC, XB1.VCC
- new net GND: C10.2, C4.2, C5.2, C6.2, C7.2, C8.2, C9.2, CN1.D-, GND_1_C1.TP, IC1.ADJ, R13.1, R17.2, R18.1, U$1.GND, U1.VSSA1, U1.VSSA2, U1.VSSD, U1.VSSIO, X1-2.KL, XB1.GND
- new net RESET_XBEE: U1.P1.6, XB1.!RESET
- new net RX_STRENGTH: U1.P1.5, XB1.RSSI/PWM/DIO10
- new net VCC_9-12V: IC1.IN, VCC_2_C1.TP, X1-1.KL
- net CANH: now also R16.2, U$1.CANH; no longer CANH_2_C1.TP, CANH_3_C1.TP, CANH_4_C1.TP, CANH_C1.TP, S1.1
- net CANL: no longer CANL_2_C1.TP, CANL_3_C1.TP, CANL_4_C1.TP, CANL_C1.TP
- net SCL_S2: no longer SCL_S2_C2.TP
- net SCL_S3: no longer SCL_S3_C3.TP
- net SDA_S2: no longer SDA_S2_C1.TP
- net SDA_S3: no longer SDA_S3_C1.TP
- net UART_RX: now also XB1.DIN/!CONFIG
- net UART_TX: now also XB1.DOUT
- net VDDA: now also L1.2; no longer VDDA_C1.TP
- net VDDD: now also L2.2; no longer VDDD_C1.TP
- net VDDIO: now also R15.2; no longer VDDIO_C1.TP
Other:
- note removed: "3V3=3.3V V. SUPPLY"
- note removed: "C?= CONNECTOR FACE 1,2,3 OR 4"
- note removed: "FACE 1 COMPONENT'S"
- note removed: "FACE 2 COMPONENT'S"
- note removed: "FACE 3 COMPONENT'S"
- note removed: "FACE 4 COMPONENT'S"
- note removed: "FACES PADS 1, 2, 3 AND 4"
- note removed: "GND=GROUND"
- note removed: "INTER FACE PADS 1,2 AND 3"
- note removed: "NODES VCC AND GROUND"
- note removed: "Soldered Only For Mechanical Purposes"
- note removed: "VCC=12V"
- moved on the sheet: C10, C4, C5, C6, C7, C8, C9, CANH_1_C1, CANL_1_C1, CRYSTAL, GND_1_C1, IC1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
