File: PCB/PCB_Eagle_mit_VCNL_V1/Robot_Psoc.brd (EAGLE design)
At the start: 235.3 x 59.5 mm, 186 parts, among them IC1 LD117AS33TR, U1 CY8C4247AZI-M485, U2 VCNL4010-GS08, U3 VCNL4010-GS08, U4 VCNL4010-GS08, U5 VCNL4010-GS08, X1 FH12-10S-0.5SH, X2 FH12-10S-0.5SH

Commit message: 16 de Enero de 2016
PCB
Parts:
- added GND_REINFORCEMENT, VCC_REINFORCEMENT: PTR1TP11R, testpad:TP11R
- moved VCC_1_C2 0.35 mm to (72.1, 69.8)
Connections:
- net GND4: now also GND_REINFORCEMENT.TP
- net VCC_C4: now also VCC_REINFORCEMENT.TP
Routing:
- net GND4: track 150.1 -> 169.4 mm, vias 3 -> 4
- net VCC_C4: track 150.0 -> 158.6 mm, vias 2 -> 3
- net VCC_C3: track 133.4 -> 137.7 mm
- net VCC_C2: track 136.2 -> 136.8 mm
Other:
- board text added: "EMERGE FACE 1"
- board text added: "EMERGE FACE 2"
- board text added: "EMERGE FACE 3"
- board text added: "EMERGE FACE 4"
