File: PCB/PCB_Eagle_mit_VCNL_V2/Robot_Psoc.brd (EAGLE design)
At the start: 222.5 x 59.5 mm, 184 parts, among them IC1 LD117AS33TR, U1 CY8C4247AZI-M485, U2 VCNL4010-GS08, U3 VCNL4010-GS08, U4 VCNL4010-GS08, U5 VCNL4010-GS08, X1 FH12-10S-0.5SH, X2 FH12-10S-0.5SH

Commit message: 16 de Enero de 2016
PCB
Parts:
- added GND_REINFORCEMENT, VCC_REINFORCEMENT: PTR1TP11R, testpad:TP11R
Connections:
- net GND4: now also GND_REINFORCEMENT.TP
- net VCC_C4: now also VCC_REINFORCEMENT.TP
Routing:
- net VCC_C4: track 115.2 -> 126.1 mm, vias 1 -> 2
- net GND4: track 136.6 -> 146.6 mm, vias 5 -> 6
- net VCC_C3: track 117.4 -> 121.7 mm
- net VCCC: track 144.8 -> 146.2 mm
- net VCC_C2: track 131.3 -> 132.3 mm
- net N$32: track 153.3 -> 152.5 mm
Other:
- board text added: "EMERGE FACE 1"
- board text added: "EMERGE FACE 2"
- board text added: "EMERGE FACE 3"
- board text added: "EMERGE FACE 4"
