File: PCB/PCB_Eagle_mit_VCNL_V2/Robot_Psoc.sch (EAGLE design)
At the start: 184 parts, among them IC1 LD117AS33TR, U1 CY8C4247AZI-M485, U2 VCNL4010-GS08, U3 VCNL4010-GS08, U4 VCNL4010-GS08, U5 VCNL4010-GS08, X1 FH12-10S-0.5SH, X2 FH12-10S-0.5SH

Commit message: 16 de Enero de 2016
PCB
Parts:
- added GND_REINFORCEMENT, VCC_REINFORCEMENT: PTR1TP11R, testpad:PTR1TP11R
Connections:
- net GND4: now also GND_REINFORCEMENT.TP
- net VCC_C4: now also VCC_REINFORCEMENT.TP
Changed lines of the file:
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@@
 <part name="CANH_4_C2" library="testpad" deviceset="TP" device="B2,54"/>
 <part name="CANH_3_C2" library="testpad" deviceset="TP" device="B2,54"/>
+<part name="VCC_REINFORCEMENT" library="testpad" deviceset="PTR1" device="TP11R"/>
+<part name="GND_REINFORCEMENT" library="testpad" deviceset="PTR1" device="TP11R"/>
 </parts>
 <sheets>
@@
 <instance part="CANH_4_C2" gate="G$1" x="187.96" y="-76.2" rot="R180"/>
 <instance part="CANH_3_C2" gate="G$1" x="187.96" y="-66.04"/>
+<instance part="VCC_REINFORCEMENT" gate="G$1" x="337.82" y="-55.88" rot="R90"/>
+<instance part="GND_REINFORCEMENT" gate="G$1" x="337.82" y="-73.66" rot="R90"/>
 </instances>
 <busses>
@@
 <junction x="335.28" y="-71.12"/>
 <label x="314.96" y="-73.66" size="1.778" layer="95"/>
+<pinref part="GND_REINFORCEMENT" gate="G$1" pin="TP"/>
+<junction x="335.28" y="-73.66"/>
 </segment>
 <segment>
@@
 <junction x="322.58" y="-55.88"/>
 <label x="312.42" y="-55.88" size="1.778" layer="95"/>
-</segment>
-<segment>
+<pinref part="VCC_REINFORCEMENT" gate="G$1" pin="TP"/>
+<junction x="335.28" y="-55.88"/>
+</segment>
+<segment>
