File: PCB/PCB_Eagle_mit_VCNL_V4/Robot_Psoc.brd (EAGLE design)
At the start: 233.4 x 55.9 mm, 205 parts, among them U1 CY8C4247AZI-M485, U2 VCNL4010-GS08, U3 VCNL4010-GS08, U4 VCNL4010-GS08, U5 VCNL4010-GS08

Commit message: 2-05-2017
Hoy
Routing:
- net MOTOR: track 72.8 -> 73.8 mm
Changed lines of the file:
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@@
 <grid distance="1" unitdist="mic" unit="mic" style="lines" multiple="1" display="no" altdistance="0.025" altunitdist="inch" altunit="inch"/>
 <layers>
-<layer number="1" name="Top" color="4" fill="1" visible="no" active="yes"/>
+<layer number="1" name="Top" color="4" fill="1" visible="yes" active="yes"/>
 <layer number="2" name="Route2" color="1" fill="3" visible="no" active="no"/>
 <layer number="3" name="Route3" color="4" fill="3" visible="no" active="no"/>
@@
 <layer number="14" name="Route14" color="1" fill="6" visible="no" active="no"/>
 <layer number="15" name="Route15" color="4" fill="6" visible="no" active="no"/>
-<layer number="16" name="Bottom" color="1" fill="1" visible="no" active="yes"/>
-<layer number="17" name="Pads" color="2" fill="1" visible="no" active="yes"/>
-<layer number="18" name="Vias" color="2" fill="1" visible="no" active="yes"/>
-<layer number="19" name="Unrouted" color="6" fill="1" visible="no" active="yes"/>
+<layer number="16" name="Bottom" color="1" fill="1" visible="yes" active="yes"/>
+<layer number="17" name="Pads" color="2" fill="1" visible="yes" active="yes"/>
+<layer number="18" name="Vias" color="2" fill="1" visible="yes" active="yes"/>
+<layer number="19" name="Unrouted" color="6" fill="1" visible="yes" active="yes"/>
 <layer number="20" name="Dimension" color="15" fill="1" visible="yes" active="yes"/>
-<layer number="21" name="tPlace" color="7" fill="1" visible="no" active="yes"/>
-<layer number="22" name="bPlace" color="7" fill="1" visible="no" active="yes"/>
-<layer number="23" name="tOrigins" color="15" fill="1" visible="no" active="yes"/>
-<layer number="24" name="bOrigins" color="15" fill="1" visible="no" active="yes"/>
-<layer number="25" name="tNames" color="7" fill="1" visible="no" active="yes"/>
-<layer number="26" name="bNames" color="7" fill="1" visible="no" active="yes"/>
-<layer number="27" name="tValues" color="7" fill="1" visible="no" active="yes"/>
-<layer number="28" name="bValues" color="7" fill="1" visible="no" active="yes"/>
-<layer number="29" name="tStop" color="7" fill="3" visible="no" active="yes"/>
-<layer number="30" name="bStop" color="7" fill="6" visible="no" active="yes"/>
-<layer number="31" name="tCream" color="7" fill="4" visible="no" active="yes"/>
-<layer number="32" name="bCream" color="7" fill="5" visible="no" active="yes"/>
-<layer number="33" name="tFinish" color="6" fill="3" visible="no" active="yes"/>
-<layer number="34" name="bFinish" color="6" fill="6" visible="no" active="yes"/>
-<layer number="35" name="tGlue" color="7" fill="4" visible="no" active="yes"/>
-<layer number="36" name="bGlue" color="7" fill="5" visible="no" active="yes"/>
-<layer number="37" name="tTest" color="7" fill="1" visible="no" active="yes"/>
-<layer number="38" name="bTest" color="7" fill="1" visible="no" active="yes"/>
+<layer number="21" name="tPlace" color="7" fill="1" visible="yes" active="yes"/>
+<layer number="22" name="bPlace" color="7" fill="1" visible="yes" active="yes"/>
+<layer number="23" name="tOrigins" color="15" fill="1" visible="yes" active="yes"/>
+<layer number="24" name="bOrigins" color="15" fill="1" visible="yes" active="yes"/>
+<layer number="25" name="tNames" color="7" fill="1" visible="yes" active="yes"/>
+<layer number="26" name="bNames" color="7" fill="1" visible="yes" active="yes"/>
+<layer number="27" name="tValues" color="7" fill="1" visible="yes" active="yes"/>
+<layer number="28" name="bValues" color="7" fill="1" visible="yes" active="yes"/>
+<layer number="29" name="tStop" color="7" fill="3" visible="yes" active="yes"/>
+<layer number="30" name="bStop" color="7" fill="6" visible="yes" active="yes"/>
+<layer number="31" name="tCream" color="7" fill="4" visible="yes" active="yes"/>
+<layer number="32" name="bCream" color="7" fill="5" visible="yes" active="yes"/>
+<layer number="33" name="tFinish" color="6" fill="3" visible="yes" active="yes"/>
+<layer number="34" name="bFinish" color="6" fill="6" visible="yes" active="yes"/>
+<layer number="35" name="tGlue" color="7" fill="4" visible="yes" active="yes"/>
+<layer number="36" name="bGlue" color="7" fill="5" visible="yes" active="yes"/>
+<layer number="37" name="tTest" color="7" fill="1" visible="yes" active="yes"/>
+<layer number="38" name="bTest" color="7" fill="1" visible="yes" active="yes"/>
 <layer number="39" name="tKeepout" color="4" fill="11" visible="no" active="yes"/>
 <layer number="40" name="bKeepout" color="1" fill="11" visible="no" active="yes"/>
@@
 <wire x1="162.287665625" y1="84.2101125" x2="161.9341125" y2="84.563665625" width="0.3048" layer="1"/>
 <wire x1="142.6076" y1="62.484" x2="140.638" y2="62.484" width="0.4064" layer="1"/>
-<wire x1="140.638" y1="62.484" x2="139.171" y2="63.951" width="0.4064" layer="1"/>
-<wire x1="139.171" y1="63.951" x2="139.171" y2="65.947" width="0.4064" layer="1"/>
-<wire x1="139.171" y1="65.947" x2="137.874" y2="67.244" width="0.4064" layer="1"/>
-<wire x1="137.874" y1="67.244" x2="126.665" y2="67.244" width="0.4064" layer="1"/>
-<wire x1="126.665" y1="67.244" x2="124.611" y2="69.298" width="0.4064" layer="1"/>
+<wire x1="126.665" y1="67.244" x2="126.375" y2="67.534" width="0.4064" layer="1"/>
+<wire x1="126.375" y1="67.534" x2="124.611" y2="69.298" width="0.4064" layer="1"/>
 <wire x1="124.611" y1="69.298" x2="124.584" y2="69.997" width="0.4064" layer="1"/>
 <via x="124.584" y="69.997" extent="1-16" drill="0.6" shape="square"/>
@@
 <wire x1="124.65" y1="80.287" x2="124.65" y2="70.407" width="0.3048" layer="16"/>
 <wire x1="124.65" y1="70.407" x2="124.584" y2="69.997" width="0.3048" layer="16"/>
+<wire x1="140.638" y1="62.484" x2="138.851" y2="62.484" width="0.6096" layer="1"/>
+<wire x1="138.851" y1="62.484" x2="138.292" y2="63.043" width="0.6096" layer="1"/>
+<wire x1="138.292" y1="63.043" x2="138.292" y2="66.145" width="0.6096" layer="1"/>
+<wire x1="138.292" y1="66.145" x2="137.152" y2="67.285" width="0.6096" layer="1"/>
+<wire x1="137.152" y1="67.285" x2="126.624" y2="67.285" width="0.6096" layer="1"/>
+<wire x1="126.624" y1="67.285" x2="126.375" y2="67.534" width="0.6096" layer="1"/>
 </signal>
 <signal name="CANH">
@@
 <wire x1="22.8782" y1="89.5298" x2="22.004" y2="88.6216" width="0.3048" layer="16"/>
 <wire x1="22.004" y1="88.6216" x2="22.04" y2="81.5884" width="0.3048" layer="16"/>
-<wire x1="22.04" y1="81.5884" x2="23.3248" y2="80.3016" width="0.3048" layer="16"/>
-<wire x1="23.3248" y1="80.3016" x2="29.0708" y2="80.2606" width="0.3048" layer="16"/>
 <via x="32.1406" y="79.6928" extent="1-16" drill="0.6" shape="square"/>
 <via x="30.2696" y="82.5518" extent="1-16" drill="0.6" shape="square"/>
@@
 <wire x1="44.893" y1="99.2268" x2="46.626" y2="100.9598" width="0.4064" layer="1"/>
 <wire x1="32.1406" y1="79.6928" x2="30.8032" y2="79.6928" width="0.4064" layer="16"/>
-<wire x1="30.8032" y1="79.6928" x2="30.24" y2="80.256" width="0.4064" layer="16"/>
-<wire x1="30.24" y1="80.256" x2="29.0754" y2="80.256" width="0.4064" layer="16"/>
-<wire x1="29.0754" y1="80.256" x2="29.0708" y2="80.2606" width="0.4064" layer="16"/>
 <wire x1="30.2696" y1="82.5518" x2="31.0032" y2="82.5518" width="0.4064" layer="1"/>
 <wire x1="31.0032" y1="82.5518" x2="32.165" y2="81.39" width="0.4064" layer="1"/>
 <wire x1="32.165" y1="81.39" x2="32.165" y2="79.7172" width="0.4064" layer="1"/>
 <wire x1="32.165" y1="79.7172" x2="32.1406" y2="79.6928" width="0.4064" layer="1"/>
+<wire x1="22.04" y1="81.5884" x2="22.04" y2="81.153" width="0.3048" layer="16"/>
+<wire x1="22.04" y1="81.153" x2="22.885" y2="80.308" width="0.3048" layer="16"/>
+<wire x1="22.885" y1="80.308" x2="30.188" y2="80.308" width="0.3048" layer="16"/>
+<wire x1="30.188" y1="80.308" x2="30.8032" y2="79.6928" width="0.3048" layer="16"/>
 </signal>
 <signal name="3V3_C4">
