File: PCB/PCB_Eagle_mit_VCNL_V4/Robot_Psoc.brd (EAGLE design)
At the start: 233.5 x 55.9 mm, 205 parts, among them U1 CY8C4247AZI-M485, U2 VCNL4010-GS08, U3 VCNL4010-GS08, U4 VCNL4010-GS08, U5 VCNL4010-GS08

Commit message: 05/May
PCB
Other:
- outline, holes or cut-outs redrawn

Commit message: 29/06/2017
Gerber
Routing:
- net 3V3_C2: track 202.6 -> 201.6 mm
- removed copper zone on layer 1, net GND_C1
Other:
- board size 233.5 x 55.9 mm -> 233.5 x 55.8 mm
