File: PCB/PCB_Eagle_Xbee_Adapter_Robot/Xbee_Adapter.sch (EAGLE design)
At the start: 34 parts, among them IC1 LD117AS33TR, U1 CY8C4247AZI-M485

Commit message: ULTIMA EDICION
Parts:
- removed IC1: LD117AS33TR, v-reg:LD117AS33TR
- removed X1: (no value), con-wago-508:W237-02P
- removed XB1: XBEE, xbee:XBEE
- added 3V3: LD117AS33TR, v-reg:LD117AS33TR
- added C2: (no value), rcl:CPOL-EUA
- added ENTRADA: (no value), con-wago-500:W237-4
- added GND_NODO, PAD1, PAD10, PAD11, PAD12, PAD13, PAD14, PAD15, PAD16, PAD17, PAD18, PAD19, PAD2, PAD20, PAD3, PAD4, PAD5, PAD6, PAD7, PAD8, PAD9, VCC_NODO: (no value), wirepad:SMD5
- added LED1, ON: (no value), adafruit:LEDCHIP-LED0805
- added R4: (no value), rcl:R-EU_R0805
- added R5: 1K, rcl:R-EU_R0805
Connections:
- new net N$10: ON.C, R5.1
- new net N$5: LED1.A, U1.P6.5
- new net N$6: LED1.C, R4.1
- new net SLEEP_CTRL: PAD9.P, U1.P1.4
- new net SLEEP_XBEE: PAD13.P, U1.P1.1
- net 3V3: now also 3V3.OUT, C2.+, ON.A, PAD1.P; no longer IC1.OUT, XB1.VCC
- net CANH: now also ENTRADA-3.KL
- net CANL: now also ENTRADA-4.KL
- net GND: now also 3V3.ADJ, C2.-, ENTRADA-2.KL, GND_NODO.P, PAD10.P, R4.2, R5.2; no longer IC1.ADJ, X1-2.KL, XB1.GND
- net RESET_XBEE: now also PAD5.P; no longer XB1.!RESET
- net RX_STRENGTH: now also PAD6.P, U1.P2.6; no longer U1.P1.5, XB1.RSSI/PWM/DIO10
- net UART_RX: now also PAD3.P, U1.P2.1/SCB1:SDA1; no longer U1.P7.0/SCB3:SCL1, XB1.DIN/!CONFIG
- net UART_TX: now also PAD2.P, U1.P2.0/SCB1:SCL1; no longer U1.P7.1/SCB3:SDA1, XB1.DOUT
- net VCC_9-12V: now also 3V3.IN, ENTRADA-1.KL, VCC_NODO.P; no longer IC1.IN, X1-1.KL
